Commit message: create storm_ros package

File: content/assets/urdf/franka_description/franka_panda_tray.urdf (robot description, URDF)
Before this commit: robot panda, 12 links, 11 joints
Links:
- link tray_link: geometry collision box size=0.245 0.25 0.04; visual box size=0.245 0.25 0.04
Joints:
- joint panda_tray_fixed_joint: origin xyz=0.0 0.1225 0.106 rpy=0.0 0.0 0.0 -> xyz=0.0 0.0 0.02 rpy=0.0 0.0 0.0

Commit message: first version of tray with orientation constraints

File: content/assets/urdf/franka_description/franka_panda_tray.urdf (robot description, URDF)
Before this commit: robot panda, 12 links, 11 joints
Links:
- link tray_link: geometry collision box size=0.25 0.245 0.04; visual box size=0.25 0.245 0.04
Joints:
- joint panda_tray_fixed_joint: origin xyz=0.0 0.0 0.02 rpy=0.0 0.0 0.0 -> xyz=0.0 0.125 0.02 rpy=0.0 0.0 0.0
