Commit message: STORM_GraspNet FrameWork

File: content/assets/urdf/franka_description/franka_panda_no_gripper.urdf (robot description, URDF)
Before this commit: robot panda, 11 links, 10 joints
Joints:
- joint ee_fixed_joint: origin xyz=0.0 0. 0.1 rpy=0.0 0.0 -1.57 -> xyz=0.0 0. 0.080 rpy=3.002 -1.469 0.109

Commit message: hold on

File: content/assets/urdf/franka_description/franka_panda_no_gripper.urdf (robot description, URDF)
Before this commit: robot panda, 11 links, 10 joints
Links:
- added link graspnet_link; collision box size=0.01 0.01 0.01
Joints:
- added joint ee_grasp_joint: type fixed, parent panda_hand, child graspnet_link, origin xyz=0.0 0. 0.080 rpy=3.002 -1.469 0.109
- joint ee_fixed_joint: origin xyz=0.0 0. 0.080 rpy=3.002 -1.469 0.109 -> xyz=0.0 0. 0.1 rpy=0.0 0.0 -1.57

File: content/assets/urdf/mug/movable_collision_test.urdf (robot description, URDF)
Before this commit: robot mug, 7 links, 6 joints
Links:
- link mug: geometry collision mesh filename=mug.obj scale=2 2 2; visual mesh filename=mug.obj scale=4 4 6
