Commit message: flip_visual_attachments=False

File: content/assets/urdf/genie_description/genieArm.urdf (robot description, URDF)
Before this commit: robot genie01, 10 links, 9 joints
Links:
- link Link1_l: geometry collision cylinder length=0.1638999544084072 radius=0.05559538401924806; visual mesh filename=meshes/visual/Link1_l.obj
- link Link2_l: geometry collision box size=0.0703125 0.08602613 0.07128906; collision box size=0.078125 0.15545113 0.021484375
- link Link3_l: geometry collision cylinder length=0.21500002965331078 radius=0.05134501389693651; visual mesh filename=meshes/visual/Link3_l.obj
- link Link4_l: geometry collision box size=0.056640625 0.07028388999999999 0.0625; collision box size=0.0703125 0.13151169 0.017578125
- link Link5_l: geometry collision cylinder length=0.12419998832046986 radius=0.04058189219799553; visual mesh filename=meshes/visual/Link5_l.obj
- link Link6_l: geometry collision box size=0.05859375 0.08339137000000002 0.05859375; collision box size=0.05859375 0.12849998 0.015625
- link Link7_l: geometry collision cylinder length=0.04599999970197749 radius=0.030803805454578115; visual mesh filename=meshes/visual/Link7_l.obj
- link Link_hand_l: geometry collision box size=0.2 0.08 0.2; collision box size=0.2 0.08 0.2
- link base_link_l: geometry collision cylinder length=0.0913499565795064 radius=0.05200000736048429; visual mesh filename=meshes/visual/base_link_l.obj

File: content/assets/urdf/genie_description/genieArmSimple.urdf (robot description, URDF)
Before this commit: robot genie01, 10 links, 9 joints
Links:
- removed link Link2_l
- removed link Link3_l
- removed link Link4_l
- removed link Link5_l
- removed link Link6_l
- removed link Link7_l
- removed link Link_hand_l
- link Link1_l: geometry collision cylinder length=0.1638999544084072 radius=0.05559538401924806; visual mesh filename=meshes/visual/Link1_l.obj
- link base_link_l: geometry collision cylinder length=0.0913499565795064 radius=0.05200000736048429; visual mesh filename=meshes/visual/base_link_l.obj
Joints:
- removed joint Joint2_l
- removed joint Joint3_l
- removed joint Joint4_l
- removed joint Joint5_l
- removed joint Joint6_l
- removed joint Joint7_l
- removed joint Joint_hand_l
