Commit message: genie-singleArm

File: content/assets/urdf/genie_description/A2DWithFixBase.urdf (robot description, URDF)
Before this commit: robot a2d_description, 25 links, 24 joints
Joints:
- joint joint_body_pitch: axis 0 0 -1 -> 0 0 1; limit lower=0 upper=1.5708 effort=100 velocity=0.5 -> lower=-1.5708 upper=0 effort=100 velocity=0.5; type fixed -> revolute
- joint joint_head_pitch: type fixed -> revolute
- joint joint_head_yaw: type fixed -> revolute
- joint joint_lift_body: type fixed -> prismatic

File: content/assets/urdf/mug/movable_collision_test.urdf (robot description, URDF)
Before this commit: robot mug, 7 links, 6 joints
Joints:
- joint x_joint: limit lower=-2 upper=2.0 effort=1 velocity=1 -> lower=-20.0 upper=20.0 effort=1 velocity=1
- joint y_joint: limit lower=-2.0 upper=2.0 effort=1 velocity=1 -> lower=-20.0 upper=20.0 effort=1 velocity=1
- joint z_joint: limit lower=-2.8973 upper=2.8973 effort=12 velocity=2.6100 -> lower=-20.0 upper=20.0 effort=1 velocity=1

Commit message: 适配dual-arm

File: content/assets/urdf/genie_description/A2DWithFixBase.urdf (robot description, URDF)
Before this commit: robot a2d_description, 25 links, 24 joints
Links:
- removed link ee_link
- added link ee_link_l
- added link ee_link_r
Joints:
- removed joint Joint_hand_damp
- added joint Joint_hand_damp_l: type fixed, parent Link_hand_l, child ee_link_l, origin xyz=0 0 0.08 rpy=0 0 0, axis 0 0 0
- added joint Joint_hand_damp_r: type fixed, parent Link_hand_r, child ee_link_r, origin xyz=0 0 0.08 rpy=0 0 0, axis 0 0 0
- joint Joint1_r: type fixed -> revolute
- joint Joint2_r: type fixed -> revolute
- joint Joint3_r: type fixed -> revolute
- joint Joint4_r: type fixed -> revolute
- joint Joint5_r: type fixed -> revolute
- joint Joint6_r: type fixed -> revolute
- joint Joint7_r: type fixed -> revolute
- joint joint_body_pitch: type revolute -> fixed
- joint joint_lift_body: limit lower=0 upper=0.555 effort=100 velocity=0.1 -> lower=0 upper=0.40 effort=100 velocity=0.1; type prismatic -> fixed

Commit message: 强化trac-ik满足双臂场景； 增加mapper的功能，统一gym, trac-ik, storm-mpc的robot model的顺序问题； 增加genie_train_self_colliison coll_val的数据加入碰撞数据与非碰撞数据，让训练曲线更平滑
Enhances dual-arm support with TRAC-IK and model unification

Refines mapper functionality to unify joint order across Gym, TRAC-IK, and Storm-MPC models, resolving inconsistencies.

Improves self-collision cost handling with smoother collision data integration for better training stability.

Adds dual-arm rollout and cost computation to support independent goal tracking for each arm, enhancing flexibility and precision in control.

Optimizes logging, debugging, and visualization for collision detection and IK results.

File: content/assets/urdf/genie_description/A2DWithFixBase.urdf (robot description, URDF)
Before this commit: robot a2d_description, 26 links, 25 joints
Joints:
- joint joint_head_pitch: type revolute -> fixed
- joint joint_head_yaw: type revolute -> fixed
