Commit message: PPV_Franka

File: content/assets/urdf/mug/movable_collision_test.urdf (robot description, URDF)
Before this commit: robot mug, 7 links, 6 joints
Links:
- link mug: geometry collision mesh filename=mug.obj scale=2 2 2; visual mesh filename=mug.obj scale=3 3 3

Commit message: print->rospy.info

File: content/assets/urdf/mug/movable_collision_test.urdf (robot description, URDF)
Before this commit: robot mug, 7 links, 6 joints
Links:
- link mug: geometry collision mesh filename=mug.obj scale=2 2 2; visual mesh filename=mug.obj scale=4 4 5

Commit message: 创新点可视化v0.0.0

File: content/assets/urdf/mug/movable_collision_test.urdf (robot description, URDF)
Before this commit: robot mug, 7 links, 6 joints
Links:
- link mug: geometry collision mesh filename=mug.obj scale=2 2 2; visual mesh filename=mug.obj scale=4.2 4.2 5.2

Commit message: 可视化v1.0

File: content/assets/urdf/mug/movable_collision_test.urdf (robot description, URDF)
Before this commit: robot mug, 7 links, 6 joints
Links:
- link mug: geometry collision mesh filename=mug.obj scale=2 2 2; visual mesh filename=mug.obj scale=3 3 4.5

Commit message: Genie_Jnc for Humanoid

File: content/assets/urdf/mug/movable_collision_test.urdf (robot description, URDF)
Before this commit: robot mug, 7 links, 6 joints
Links:
- link mug: geometry collision mesh filename=mug.obj scale=2 2 2; visual cylinder length=0.4 radius=0.16
